Commit message: update practice3_urdf,joints can work correctly

File: install/practice3_urdf/share/practice3_urdf/practice3/urdf/practice3.urdf (robot description, URDF)
Before this commit: robot practice3_urdf, 9 links, 8 joints
Links:
- link R_Hip_Link: mass 0 -> 0.337321088171608
Joints:
- joint L_Hip_Joint: axis 0 0 -1 -> 0.997103255683817 0 -0.0760598284558406; origin xyz=-0.057 0.18415 0 rpy=0 -0.076133 -3.1416 -> xyz=0.18415 0.0569999999999967 0.202799999999937 rpy=0 -0.0761333556172417 1.5707963267949
- joint L_Knee_Joint: axis 0 0 1 -> 0 0.347852975024765 0.937549096189858
- joint L_Wheel_Joint: axis 0 0 1 -> 0 0.577491348313505 -0.816396804637947
- joint R_Hip_Joint: axis 0 0 1 -> 0.539707068979717 0 -0.841852884828058; origin xyz=-0.22448 -0.18865 -0.086956 rpy=3.1416 1.0007 0 -> xyz=-0.188649999999999 0.224484620762522 0.115844278991675 rpy=3.14159265358979 1.00070721609115 -1.5707963267949
- joint R_Knee_Joint: axis 0 0 1 -> 0 0.55876909327944 -0.829323278580598
- joint R_Wheel_Joint: axis 0 0 1 -> 0 0.577491348313505 -0.816396804637947

File: install/practice3_urdf/share/practice3_urdf/urdf/practice3.urdf (robot description, URDF)
Before this commit: robot practice3, 9 links, 8 joints
Links:
- removed link L_Ankle_Link
- removed link R_Ankle_Link
- link L_Hip_Link: mass 0.344128323066193 -> 0.34413
- link L_Knee_Link: mass 0.302555540985452 -> 0.30256
- link L_Wheel_Link: mass 0.227350411005584 -> 0.22735
- link R_Hip_Link: mass 0.337321088171608 -> 0.33732
- link R_Knee_Link: mass 0.302555410163473 -> 0.30256
- link R_Wheel_Link: mass 0.227350411005584 -> 0.19406
- link base_link: mass 10.1429242656751 -> 8.3728
Joints:
- removed joint L_Ankle_Joint
- removed joint R_Ankle_Joint
- joint L_Hip_Joint: axis 0.997103255683817 0 -0.0760598284558406 -> 0 0 -1; limit lower=0 upper=0 effort=0 velocity=0 -> lower=3.14 upper=0 effort=0 velocity=0; origin xyz=0.18415 0.0569999999999967 0.202799999999937 rpy=0 -0.0761333556172417 1.5707963267949 -> xyz=-0.057 0.16105 0 rpy=1.5708 1.5046 -3.1416
- joint L_Knee_Joint: axis 0 0.347852975024765 0.937549096189858 -> 0 0 1; origin xyz=-0.201693335514952 0.0156000000000005 -0.16999156630502 rpy=1.84994305906754 0 -1.5707963267949 -> xyz=0.17 0 0 rpy=0 0 -1.5608
- joint L_Wheel_Joint: axis 0 0.577491348313505 -0.816396804637947 -> 0 0 1; origin xyz=0.039499999996716 0 0 rpy=-0.970932593051184 0 0 -> xyz=0.2 0 0.0373 rpy=0 0 3.0655; parent L_Ankle_Link -> L_Knee_Link
- joint R_Hip_Joint: axis 0.539707068979717 0 -0.841852884828058 -> 0 0 1; origin xyz=-0.188649999999999 0.224484620762522 0.115844278991675 rpy=3.14159265358979 1.00070721609115 -1.5707963267949 -> xyz=-0.057 -0.16105 0 rpy=1.5708 0.60989 -3.1416
- joint R_Knee_Joint: axis 0 0.55876909327944 -0.829323278580598 -> 0 0 1; origin xyz=0.183638766649337 -0.0200999999999994 -0.138480335728618 rpy=1.97860271658443 0 1.5707963267949 -> xyz=0.17 0 0 rpy=0 0 -2.1771
- joint R_Wheel_Joint: axis 0 0.577491348313505 -0.816396804637947 -> 0 0 1; origin xyz=0.0395 0 0 rpy=-0.027332 0 0 -> xyz=0.2 0 -0.0373 rpy=0 0 2.787; parent R_Ankle_Link -> R_Knee_Link
